File: pcb/_autosave-pcb.kicad_sch (KiCad schematic)
At the start: 22 parts, among them J1 Conn_Coaxial_Power, J2 AudioJack3, U1 TDA7294

Commit message: Doc conception schéma complétée
Parts:
- J2: footprint Connector_Audio:Jack_3.5mm_CUI_SJ1-3523N_Horizontal -> (none)
Changed lines of the file:
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@@
 			)
 		)
-		(property "Footprint" "Connector_Audio:Jack_3.5mm_CUI_SJ1-3523N_Horizontal"
+		(property "Footprint" ""
 			(at 86.36 99.06 0)
 			(effects

Commit message: Update PCB
Parts:
- J2: footprint (none) -> Connector_Audio:Jack_3.5mm_CUI_SJ1-3523N_Horizontal
Changed lines of the file:
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@@
 			)
 		)
-		(property "Footprint" ""
+		(property "Footprint" "Connector_Audio:Jack_3.5mm_CUI_SJ1-3523N_Horizontal"
 			(at 86.36 99.06 0)
 			(effects
