File: pcb/pcb.kicad_pcb (KiCad board)
At the start: 2 copper layers, 21 parts, among them J1 Conn_Coaxial_Power, U1 TDA7294

Commit message: Update PCB
Parts:
- added J2: AudioJack3, Connector_Audio:Jack_3.5mm_CUI_SJ1-3523N_Horizontal, F.Cu at (89.5, 83.5)
- moved C9 6.75 mm to (100.5, 98.5)
- moved R3 5.50 mm to (91.4, 111.5)
- moved C8 4.98 mm to (105.5, 69.0)
- moved R2 4.50 mm to (91.4, 117.5)
- moved C5 3.50 mm to (91.5, 124.0)
Connections:
- net - renamed Net-(J1-Ext)
- C2 pad 1: + -> Net-(J1-In)
- C4 pad 1: Net-(J1-In) -> Net-(C4-Pad1)
- C7 pad 1: + -> Net-(J1-In)
- R1 pad 1: + -> Net-(J1-In)
- R6 pad 1: + -> Net-(J1-In)
- U1 pad 13: + -> Net-(J1-In)
- U1 pad 7: + -> Net-(J1-In)
Routing:
- net +: track 77.8 -> 0.00 mm, vias 1 -> 0
- net Net-(J1-In): track 44.3 -> 113.8 mm
- net Net-(C4-Pad1): track 0.00 -> 34.3 mm, vias 0 -> 2
- net GND: track 173.5 -> 198.5 mm
- net Net-(U1-STBY): track 50.8 -> 59.1 mm
- net Net-(U1-+): track 14.8 -> 20.3 mm
- net Net-(D1-A): track 70.1 -> 64.9 mm
- net Net-(U1--): track 27.6 -> 32.1 mm
- net Net-(C5-Pad1): track 7.55 -> 6.55 mm
Other:
- board outline added: 77.5 x 70 mm

Commit message: Update PCB & recherches
Parts:
- moved C4 0.59 mm to (109.0, 99.5), turned to 0 degrees
Routing:
- net Net-(C4-Pad1): track 34.3 -> 19.6 mm
- net Net-(U1--): track 32.1 -> 45.1 mm
- net Net-(D1-A): track 64.9 -> 53.9 mm, vias 0 -> 1
- net Net-(J1-In): track 113.8 -> 105.8 mm, vias 2 -> 1
- net GND: track 198.5 -> 204.9 mm, vias 0 -> 1
- net Net-(U1-BOOT): track 28.5 -> 31.0 mm
- net Net-(C10-Pad2): track 48.5 -> 50.8 mm
- net Net-(U1-STBY): track 59.1 -> 57.0 mm, vias 0 -> 1
- net Net-(J1-Ext): track 49.1 -> 50.4 mm
- net Net-(C5-Pad1): track 6.55 -> 7.22 mm

Commit message: doc création pcb terminée
Routing:
- net Net-(C4-Pad1): track 19.6 -> 30.9 mm
Changed lines of the file:
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@@
 		(tags "capacitor handsolder")
 		(property "Reference" "C4"
-			(at 0 -1.85 360)
+			(at 0 -1.85 0)
 			(layer "F.SilkS")
 			(effects
@@
 		)
 		(property "Value" "470N"
-			(at 0 1.85 360)
+			(at 0 1.85 0)
 			(layer "F.Fab")
 			(effects
@@
 		)
 		(fp_text user "${REFERENCE}"
-			(at 0 0 360)
+			(at 0 0 0)
 			(layer "F.Fab")
 			(effects
@@
 	)
 	(segment
+		(start 96 80)
+		(end 94.5 78.5)
+		(width 0.25)
+		(layer "F.Cu")
+		(net 4)
+	)
+	(segment
 		(start 107.4375 99.5)
 		(end 107.4375 96.6875)
@@
 	)
 	(segment
+		(start 94.5 88.5)
+		(end 96 87)
+		(width 0.25)
+		(layer "F.Cu")
+		(net 4)
+	)
+	(segment
 		(start 95 88.5)
 		(end 94.5 88.5)
@@
 	)
 	(segment
+		(start 96 87)
+		(end 96 80)
+		(width 0.25)
+		(layer "F.Cu")
+		(net 4)
+	)
+	(segment
 		(start 99.25 88.5)
 		(end 94.5 88.5)
@@
 	)
 	(segment
-		(start 132.5 87)
-		(end 132.5 84)
-		(width 0.5)
-		(layer "F.Cu")
-		(net 8)
-	)
-	(segment
 		(start 128 80.62)
 		(end 132.06 76.56)
@@
 	)
 	(segment
+		(start 132.5 87)
+		(end 132.5 84)
+		(width 0.5)
+		(layer "F.Cu")
+		(net 8)
+	)
+	(segment
 		(start 132.06 76.56)
 		(end 133.25 76.56)
@@
 	(via
 		(at 132.5 84)
-		(size 0.5)
-		(drill 0.25)
+		(size 0.6)
+		(drill 0.3)
 		(layers "F.Cu" "B.Cu")
 		(net 8)
@@
 	)
 	(segment
-		(start 112 101.75)
+		(start 111.88 105.5)
 		(end 112 105.38)
 		(width 0.5)
@@
 	(segment
 		(start 112 105.38)
-		(end 111.88 105.5)
+		(end 112 101.75)
 		(width 0.5)
 		(layer "F.Cu")
@@
 	(via
 		(at 112 101.75)
-		(size 0.5)
-		(drill 0.25)
+		(size 0.6)
+		(drill 0.3)
 		(layers "F.Cu" "B.Cu")
 		(net 13)
